File: projet_escape_game.kicad_pcb (KiCad board)
At the start: 2 copper layers, 71 x 70.5 mm, 41 parts, among them J1 Conn_01x03_Pin, J2 Conn_02x07_Odd_Even, J3 Conn_OLED_Display, J4 Conn_01x02, M2 RFID-RC522, SW1 SW_SPST, SW2 SW_SPST, SW3 SW_SPST, SW4 SW_SPST, U1 STM32L021K4Tx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

Commit message: Add files via upload
Routing:
- net SWDCK: track 43.3 -> 46.9 mm
- net SWDIO: track 38.9 -> 41.7 mm
- net Button1: track 63.2 -> 61.9 mm
- net GND: track 10.6 -> 11.5 mm
Other:
- board text added: "TEAM Brutier"
- board text removed: "TEAM B"
